File: pcb/LCD-BackPack_v11.sch (EAGLE design)
At the start: 70 parts, among them IC1 MEGA328, J1 AVR_SPI, P1 VSS, P10 DB3, P11 DB4, P12 DB5, P13 DB6, P14 DB7, P15 BL(+), P16 BL(-), P17 BL(-), P18 BL(-), P19 VSS, P2 VDD, P20 VDD, P21 VE, P22 RS, P23 R/W, P24 EN, P25 DB0, P26 DB1, P27 DB2, P28 DB3, P29 DB4, P3 VE, P30 DB5, P31 DB6, P32 DB7, P33 BL(+), P34 BL(-), P4 RS, P5 R/W, P6 EN, P7 DB0, P8 DB1, P9 DB2, Y1 16MHz

Commit message: cleaned up schematics and layout
Changed lines of the file:
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@@
 <setting verticaltext="up"/>
 </settings>
-<grid distance="0.1" unitdist="inch" unit="inch" style="lines" multiple="1" display="no" altdistance="0.01" altunitdist="inch" altunit="inch"/>
+<grid distance="0.05" unitdist="inch" unit="inch" style="lines" multiple="1" display="yes" altdistance="0.025" altunitdist="inch" altunit="inch"/>
 <layers>
 <layer number="1" name="Top" color="4" fill="1" visible="no" active="no"/>
@@
 <part name="T2" library="zetex" deviceset="NMOSSOT23" device=""/>
 <part name="T3" library="zetex" deviceset="NMOSSOT23" device=""/>
-<part name="FRAME2" library="frames" deviceset="A4L-LOC" device=""/>
+<part name="FRAME1" library="we-symbol" deviceset="FRAME-A4L" device=""/>
 </parts>
 <sheets>
@@
 <text x="117.475" y="114.935" size="1.778" layer="91">TXD</text>
 <text x="117.475" y="117.475" size="1.778" layer="91">RXD</text>
-<text x="161.29" y="31.75" size="1.27" layer="95">Released under the Creative Commons Attribution Share-Alike License</text>
-<text x="161.29" y="29.21" size="1.27" layer="95">http://creativecommons.org/licenses/by-sa/4.0/</text>
-<text x="161.29" y="25.4" size="1.27" layer="95">Designed by Aleksej Lazarev (Watterott electronic)</text>
+<text x="162.56" y="21.59" size="1.27" layer="95">Released under the Creative Commons Attribution Share-Alike License</text>
+<text x="162.56" y="19.05" size="1.27" layer="95">http://creativecommons.org/licenses/by-sa/4.0/</text>
+<text x="162.56" y="15.24" size="1.27" layer="95">Designed by Aleksej Lazarev (Watterott electronic)</text>
 <wire x1="172.085" y1="128.27" x2="172.085" y2="126.365" width="0.8128" layer="94"/>
 <wire x1="168.91" y1="153.67" x2="168.91" y2="151.765" width="0.8128" layer="94"/>
@@
 <instance part="C8" gate="G$1" x="215.265" y="151.13" rot="R90"/>
 <instance part="GND19" gate="1" x="46.99" y="30.48" rot="R90"/>
-<instance part="U$1" gate="G$1" x="204.47" y="19.05"/>
-<instance part="LOGO1" gate="G$1" x="204.47" y="11.43"/>
+<instance part="U$1" gate="G$1" x="208.28" y="7.62"/>
+<instance part="LOGO1" gate="G$1" x="198.12" y="7.62"/>
 <instance part="T1" gate="A" x="191.135" y="45.72"/>
 <instance part="T2" gate="A" x="191.135" y="63.5"/>
 <instance part="T3" gate="A" x="191.135" y="81.28"/>
-<instance part="FRAME2" gate="G$1" x="0" y="0"/>
+<instance part="FRAME1" gate="G$1" x="0" y="0"/>
 </instances>
 <busses>
